File: LED-display.sch (KiCad schematic (older format))
At the start: 85 parts, among them J1 Conn_01x01_Male, J10 Conn_01x01_Male, J11 Conn_01x01_Male, J12 Conn_01x01_Male, J13 Conn_01x01_Male, J14 Conn_01x01_Male, J2 Conn_01x01_Male, J3 Conn_01x01_Male, J4 Conn_01x01_Male, J5 Conn_01x01_Male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

Commit message: Move buttons
Parts:
- added MH1, MH2, MH3, MH4: MountingHole, MountingHole:MountingHole_5.5mm, symbol Mechanical:MountingHole
Changed lines of the file:
@@
 Wire Wire Line
 	2650 4500 2750 4500
+$Comp
+L Mechanical:MountingHole MH1
+U 1 1 5D12FF79
+P 13000 5000
+F 0 "MH1" H 13100 5046 50  0000 L CNN
+F 1 "MountingHole" H 13100 4955 50  0000 L CNN
+F 2 "MountingHole:MountingHole_5.5mm" H 13000 5000 50  0001 C CNN
+F 3 "~" H 13000 5000 50  0001 C CNN
+	1    13000 5000
+	1    0    0    -1
+$EndComp
+$Comp
+L Mechanical:MountingHole MH2
+U 1 1 5D1301DF
+P 13000 5300
+F 0 "MH2" H 13100 5346 50  0000 L CNN
+F 1 "MountingHole" H 13100 5255 50  0000 L CNN
+F 2 "MountingHole:MountingHole_5.5mm" H 13000 5300 50  0001 C CNN
+F 3 "~" H 13000 5300 50  0001 C CNN
+	1    13000 5300
+	1    0    0    -1
+$EndComp
+$Comp
+L Mechanical:MountingHole MH3
+U 1 1 5D1302D7
+P 13000 5600
+F 0 "MH3" H 13100 5646 50  0000 L CNN
+F 1 "MountingHole" H 13100 5555 50  0000 L CNN
+F 2 "MountingHole:MountingHole_5.5mm" H 13000 5600 50  0001 C CNN
+F 3 "~" H 13000 5600 50  0001 C CNN
+	1    13000 5600
+	1    0    0    -1
+$EndComp
+$Comp
+L Mechanical:MountingHole MH4
+U 1 1 5D1303C9
+P 13000 5900
+F 0 "MH4" H 13100 5946 50  0000 L CNN
+F 1 "MountingHole" H 13100 5855 50  0000 L CNN
+F 2 "MountingHole:MountingHole_5.5mm" H 13000 5900 50  0001 C CNN
+F 3 "~" H 13000 5900 50  0001 C CNN
+	1    13000 5900
+	1    0    0    -1
+$EndComp
 $EndSCHEMATC

Commit message: Small fixes
Parts:
- removed R46, R47, R48, R49: 0, Resistor_SMD:R_0805_2012Metric_Pad1.15x1.40mm_HandSolder, symbol Device:R
- added J15: PWM, Connector_PinHeader_2.54mm:PinHeader_1x01_P2.54mm_Vertical, symbol Connector:Conn_01x01_Male
- J1: value Conn_01x01_Male -> Data
- J11: value Conn_01x01_Male -> Gnd
- J12: value Conn_01x01_Male -> Vcc
- J2: value Conn_01x01_Male -> Clock
- J3: value Conn_01x01_Male -> Latch
Connections:
- net labels added: PWM
- wire segments 258 -> 259
Changed lines of the file:
@@
 	3150 2950 3150 3050
-$Comp
-L MyLib:TPIC6C595 D2
-U 1 1 5CD6AF2E
-P 3150 4350
-F 0 "D2" H 2900 4950 50  0000 C CNN
-F 1 "TPIC6C595" H 3400 4950 50  0000 C CNN
-F 2 "Package_SO:SOIC-16_3.9x9.9mm_P1.27mm" H 3550 3900 50  0001 C CNN
-F 3 "" H 3550 3900 50  0001 C CNN
-	1    3150 4350
-	1    0    0    -1
-$EndComp
 $Comp
 L MyLib:White7seg HL2
@@
 	3150 8950 3150 9050
 $Comp
-L power:GND #PWR0113
-U 1 1 5CDB777F
-P 2600 2800
-F 0 "#PWR0113" H 2600 2550 50  0001 C CNN
-F 1 "GND" H 2605 2627 50  0000 C CNN
-F 2 "" H 2600 2800 50  0001 C CNN
-F 3 "" H 2600 2800 50  0001 C CNN
-	1    2600 2800
-	1    0    0    -1
-$EndComp
-$Comp
 L Connector:Conn_01x01_Male J1
 U 1 1 5CDF2B3E
 P 1050 7850
 F 0 "J1" H 1250 7900 50  0000 C CNN
-F 1 "Conn_01x01_Male" H 800 7900 50  0000 C CNN
+F 1 "Data" H 800 7900 50  0000 C CNN
 F 2 "Connector_PinHeader_2.54mm:PinHeader_1x01_P2.54mm_Vertical" H 1050 7850 50  0001 C CNN
 F 3 "~" H 1050 7850 50  0001 C CNN
@@
 P 900 2050
 F 0 "J2" H 1100 2100 50  0000 C CNN
-F 1 "Conn_01x01_Male" H 650 2100 50  0000 C CNN
+F 1 "Clock" H 650 2100 50  0000 C CNN
 F 2 "Connector_PinHeader_2.54mm:PinHeader_1x01_P2.54mm_Vertical" H 900 2050 50  0001 C CNN
 F 3 "~" H 900 2050 50  0001 C CNN
@@
 P 900 2350
 F 0 "J3" H 1100 2400 50  0000 C CNN
-F 1 "Conn_01x01_Male" H 650 2400 50  0000 C CNN
+F 1 "Latch" H 650 2400 50  0000 C CNN
 F 2 "Connector_PinHeader_2.54mm:PinHeader_1x01_P2.54mm_Vertical" H 900 2350 50  0001 C CNN
 F 3 "~" H 900 2350 50  0001 C CNN
@@
 P 12000 2100
 F 0 "J11" H 12106 2278 50  0000 C CNN
-F 1 "Conn_01x01_Male" H 11900 2050 50  0000 C CNN
+F 1 "Gnd" H 11900 2050 50  0000 C CNN
 F 2 "Connector_PinHeader_2.54mm:PinHeader_1x01_P2.54mm_Vertical" H 12000 2100 50  0001 C CNN
 F 3 "~" H 12000 2100 50  0001 C CNN
@@
 P 13350 2100
 F 0 "J12" H 13323 2123 50  0000 R CNN
-F 1 "Conn_01x01_Male" H 13450 2050 50  0000 R CNN
+F 1 "Vcc" H 13450 2050 50  0000 R CNN
 F 2 "Connector_PinHeader_2.54mm:PinHeader_1x01_P2.54mm_Vertical" H 13350 2100 50  0001 C CNN
 F 3 "~" H 13350 2100 50  0001 C CNN
@@
 Text Label 1350 7850 0    50   ~ 0
 Data
-$Comp
-L Device:R R46
-U 1 1 5CD7FEE3
-P 2600 2600
-F 0 "R46" H 2670 2646 50  0000 L CNN
-F 1 "0" H 2670 2555 50  0000 L CNN
-F 2 "Resistor_SMD:R_0805_2012Metric_Pad1.15x1.40mm_HandSolder" V 2530 2600 50  0001 C CNN
-F 3 "~" H 2600 2600 50  0001 C CNN
-	1    2600 2600
-	1    0    0    -1
-$EndComp
-Wire Wire Line
-	2600 2750 2600 2800
 Wire Wire Line
 	2600 2450 2750 2450
-$Comp
-L power:GND #PWR0114
-U 1 1 5CDA58A3
-P 2650 4850
-F 0 "#PWR0114" H 2650 4600 50  0001 C CNN
-F 1 "GND" H 2655 4677 50  0000 C CNN
-F 2 "" H 2650 4850 50  0001 C CNN
-F 3 "" H 2650 4850 50  0001 C CNN
-	1    2650 4850
-	1    0    0    -1
-$EndComp
-$Comp
-L Device:R R47
-U 1 1 5CDA58A9
-P 2650 4650
-F 0 "R47" H 2720 4696 50  0000 L CNN
-F 1 "0" H 2720 4605 50  0000 L CNN
-F 2 "Resistor_SMD:R_0805_2012Metric_Pad1.15x1.40mm_HandSolder" V 2580 4650 50  0001 C CNN
-F 3 "~" H 2650 4650 50  0001 C CNN
-	1    2650 4650
-	1    0    0    -1
-$EndComp
-Wire Wire Line
-	2650 4800 2650 4850
-$Comp
-L power:GND #PWR0115
-U 1 1 5CDCB1A1
-P 2650 6800
-F 0 "#PWR0115" H 2650 6550 50  0001 C CNN
-F 1 "GND" H 2655 6627 50  0000 C CNN
-F 2 "" H 2650 6800 50  0001 C CNN
-F 3 "" H 2650 6800 50  0001 C CNN
-	1    2650 6800
-	1    0    0    -1
-$EndComp
-$Comp
-L Device:R R48
-U 1 1 5CDCB1A7
-P 2650 6600
-F 0 "R48" H 2720 6646 50  0000 L CNN
-F 1 "0" H 2720 6555 50  0000 L CNN
-F 2 "Resistor_SMD:R_0805_2012Metric_Pad1.15x1.40mm_HandSolder" V 2580 6600 50  0001 C CNN
-F 3 "~" H 2650 6600 50  0001 C CNN
-	1    2650 6600
-	1    0    0    -1
-$EndComp
-Wire Wire Line
-	2650 6750 2650 6800
-$Comp
-L power:GND #PWR0116
-U 1 1 5CDDDEA6
-P 2650 8800
-F 0 "#PWR0116" H 2650 8550 50  0001 C CNN
-F 1 "GND" H 2655 8627 50  0000 C CNN
-F 2 "" H 2650 8800 50  0001 C CNN
-F 3 "" H 2650 8800 50  0001 C CNN
-	1    2650 8800
-	1    0    0    -1
-$EndComp
-$Comp
-L Device:R R49
-U 1 1 5CDDDEAC
-P 2650 8600
-F 0 "R49" H 2720 8646 50  0000 L CNN
-F 1 "0" H 2720 8555 50  0000 L CNN
-F 2 "Resistor_SMD:R_0805_2012Metric_Pad1.15x1.40mm_HandSolder" V 2580 8600 50  0001 C CNN
-F 3 "~" H 2650 8600 50  0001 C CNN
-	1    2650 8600
-	1    0    0    -1
-$EndComp
-Wire Wire Line
-	2650 8750 2650 8800
-Wire Wire Line
-	2650 8450 2750 8450
-Wire Wire Line
-	2650 6450 2750 6450
-Wire Wire Line
-	2650 4500 2750 4500
 $Comp
 L Mechanical:MountingHole MH1
@@
 	1    0    0    -1
 $EndComp
+$Comp
+L MyLib:TPIC6C595 D2
+U 1 1 5CD6AF2E
+P 3150 4350
+F 0 "D2" H 2900 4950 50  0000 C CNN
+F 1 "TPIC6C595" H 3400 4950 50  0000 C CNN
+F 2 "Package_SO:SOIC-16_3.9x9.9mm_P1.27mm" H 3550 3900 50  0001 C CNN
+F 3 "" H 3550 3900 50  0001 C CNN
+	1    3150 4350
+	1    0    0    -1
+$EndComp
+$Comp
+L Connector:Conn_01x01_Male J15
+U 1 1 5D31F837
+P 900 2600
+F 0 "J15" H 1100 2700 50  0000 C CNN
+F 1 "PWM" H 650 2650 50  0000 C CNN
+F 2 "Connector_PinHeader_2.54mm:PinHeader_1x01_P2.54mm_Vertical" H 900 2600 50  0001 C CNN
+F 3 "~" H 900 2600 50  0001 C CNN
+	1    900  2600
+	1    0    0    -1
+$EndComp
+Wire Wire Line
+	2600 4500 2750 4500
+Wire Wire Line
+	2600 2450 2600 2600
+Wire Wire Line
+	1100 2600 2600 2600
+Connection ~ 2600 2600
+Wire Wire Line
+	2600 2600 2600 4500
+Wire Wire Line
+	2600 6450 2750 6450
+Connection ~ 2600 4500
+Wire Wire Line
+	2600 4500 2600 6450
+Wire Wire Line
+	2600 8450 2750 8450
+Connection ~ 2600 6450
+Wire Wire Line
+	2600 6450 2600 8450
+Text Label 1250 2600 0    50   ~ 0
+PWM
 $EndSCHEMATC

Commit message: Now it's double side pcb
Parts:
- added J16: Conn_01x01_Male, Connector_PinHeader_2.54mm:PinHeader_1x01_P2.54mm_Vertical, symbol Connector:Conn_01x01_Male
- added R46: R, Resistor_SMD:R_0805_2012Metric_Pad1.15x1.40mm_HandSolder, symbol Device:R
- added R47: R_PHOTO, OptoDevice:R_LDR_4.9x4.2mm_P2.54mm_Vertical, symbol Device:R_PHOTO
Connections:
- wire segments 259 -> 264
Changed lines of the file:
@@
 Text Label 1250 2600 0    50   ~ 0
 PWM
+$Comp
+L Device:R_PHOTO R47
+U 1 1 5D399AA0
+P 11400 5850
+F 0 "R47" H 11470 5896 50  0000 L CNN
+F 1 "R_PHOTO" H 11470 5805 50  0000 L CNN
+F 2 "OptoDevice:R_LDR_4.9x4.2mm_P2.54mm_Vertical" V 11450 5600 50  0001 L CNN
+F 3 "~" H 11400 5800 50  0001 C CNN
+	1    11400 5850
+	1    0    0    -1
+$EndComp
+$Comp
+L Device:R R46
+U 1 1 5D399BBA
+P 11400 5350
+F 0 "R46" H 11470 5396 50  0000 L CNN
+F 1 "R" H 11470 5305 50  0000 L CNN
+F 2 "Resistor_SMD:R_0805_2012Metric_Pad1.15x1.40mm_HandSolder" V 11330 5350 50  0001 C CNN
+F 3 "~" H 11400 5350 50  0001 C CNN
+	1    11400 5350
+	1    0    0    -1
+$EndComp
+$Comp
+L power:GND #PWR021
+U 1 1 5D399D6A
+P 11400 6100
+F 0 "#PWR021" H 11400 5850 50  0001 C CNN
+F 1 "GND" H 11405 5927 50  0000 C CNN
+F 2 "" H 11400 6100 50  0001 C CNN
+F 3 "" H 11400 6100 50  0001 C CNN
+	1    11400 6100
+	1    0    0    -1
+$EndComp
+$Comp
+L power:VCC #PWR020
+U 1 1 5D39A336
+P 11400 5050
+F 0 "#PWR020" H 11400 4900 50  0001 C CNN
+F 1 "VCC" H 11417 5223 50  0000 C CNN
+F 2 "" H 11400 5050 50  0001 C CNN
+F 3 "" H 11400 5050 50  0001 C CNN
+	1    11400 5050
+	1    0    0    -1
+$EndComp
+Wire Wire Line
+	11400 5050 11400 5200
+Wire Wire Line
+	11400 5500 11400 5600
+Wire Wire Line
+	11400 6000 11400 6100
+$Comp
+L Connector:Conn_01x01_Male J16
+U 1 1 5D3D4284
+P 11050 5600
+F 0 "J16" H 11156 5778 50  0000 C CNN
+F 1 "Conn_01x01_Male" H 11156 5687 50  0000 C CNN
+F 2 "Connector_PinHeader_2.54mm:PinHeader_1x01_P2.54mm_Vertical" H 11050 5600 50  0001 C CNN
+F 3 "~" H 11050 5600 50  0001 C CNN
+	1    11050 5600
+	1    0    0    -1
+$EndComp
+Wire Wire Line
+	11250 5600 11400 5600
+Connection ~ 11400 5600
+Wire Wire Line
+	11400 5600 11400 5700
 $EndSCHEMATC

Commit message: Enlarge holes and pads. Fix pinheader pos.
Parts:
- MH1, MH2, MH3, MH4: footprint MountingHole:MountingHole_5.5mm -> MountingHole:MountingHole_6mm
Changed lines of the file:
@@
 F 0 "MH1" H 13100 5046 50  0000 L CNN
 F 1 "MountingHole" H 13100 4955 50  0000 L CNN
-F 2 "MountingHole:MountingHole_5.5mm" H 13000 5000 50  0001 C CNN
+F 2 "MountingHole:MountingHole_6mm" H 13000 5000 50  0001 C CNN
 F 3 "~" H 13000 5000 50  0001 C CNN
 	1    13000 5000
@@
 F 0 "MH2" H 13100 5346 50  0000 L CNN
 F 1 "MountingHole" H 13100 5255 50  0000 L CNN
-F 2 "MountingHole:MountingHole_5.5mm" H 13000 5300 50  0001 C CNN
+F 2 "MountingHole:MountingHole_6mm" H 13000 5300 50  0001 C CNN
 F 3 "~" H 13000 5300 50  0001 C CNN
 	1    13000 5300
@@
 F 0 "MH3" H 13100 5646 50  0000 L CNN
 F 1 "MountingHole" H 13100 5555 50  0000 L CNN
-F 2 "MountingHole:MountingHole_5.5mm" H 13000 5600 50  0001 C CNN
+F 2 "MountingHole:MountingHole_6mm" H 13000 5600 50  0001 C CNN
 F 3 "~" H 13000 5600 50  0001 C CNN
 	1    13000 5600
@@
 F 0 "MH4" H 13100 5946 50  0000 L CNN
 F 1 "MountingHole" H 13100 5855 50  0000 L CNN
-F 2 "MountingHole:MountingHole_5.5mm" H 13000 5900 50  0001 C CNN
+F 2 "MountingHole:MountingHole_6mm" H 13000 5900 50  0001 C CNN
 F 3 "~" H 13000 5900 50  0001 C CNN
 	1    13000 5900
